File: hw/Pletacka_board.sch (EAGLE design)
At the start: 47 parts, among them U1 LM75BDP, U2 EL357N(A)(TA)-G, U3 EL357N(A)(TA)-G, U4 EL357N(A)(TA)-G, U5 EL357N(A)(TA)-G, U6 TPS54231D

Commit message: Fix Cednik's issues
Parts:
- added D2, D4, D6: B5819W, B5819W:B5819W
- added D3: SS34, diode:SHOTTKY-SMA
- added JP3: (no value), pinhead:PINHD-1X4
- C1: value 10u -> 10u/50V; device rcl_upravena:C-EUC0603 -> rcl_upravena:C-EUC1206; LSCS_ID C19702 -> C13585
- C4, C5: value 1u -> 100n; LCSC_ID C15849 -> C14663
- R10, R12, R6, R8: value 1k -> 2k/0.25W; device rcl_upravena:R-EU_R0603 -> rcl_upravena:R-EU_R1206; LSCS_ID C21190 -> C17944
- U1: value LM75BDP -> LM75BDP-NEW; device LM75BDP:LM75BDP -> LM75BDP:LM75BDP-NEW
Connections:
- net GND: now also D3.A, JP3.1, JP3.2, JP3.3, JP3.4; no longer D1.A
- net N$14: now also D1.A
- net N$15: now also D1.C
- net N$17: now also D2.A
- net N$18: now also D2.C
- net N$20: now also D4.A
- net N$21: now also D4.C
- net N$7: now also D6.A
- net N$9: now also D6.C
- net PH: now also D3.C; no longer D1.C
Other:
- moved on the sheet: CON1-1, CON1-2, CON2-1, CON2-2, CON3-1, CON3-2, CON4-1, CON4-2, R10, R12, R6, R8
