File: hw/Buttons.sch (KiCad schematic (older format))
At the start: 9 parts, among them SW1 SW_Push_Dual_x2, SW2 SW_Push_Dual_x2, SW3 SW_Push_Dual_x2

Commit message: Update some packages, add 3D models
Parts:
- C1, C2, C3: LCSC_ID (none) -> C14663
- R1, R2, R3: LCSC_ID (none) -> C4190
- SW1, SW2: footprint Button_Switch_SMD:SW_SPST_SKQG_WithStem -> Button_SMD:SW_SPST_SKQG_WithStem; LCSC_ID (none) -> C318887
- SW3: footprint Resistor_SMD:R_0603_1608Metric -> Button_SMD:SW_SPST_SKQG_WithStem; LCSC_ID (none) -> C318887
Changed lines of the file:
@@
 F 0 "SW1" H 5900 2635 50  0000 C CNN
 F 1 "SW_Push_Dual_x2" H 5900 2544 50  0000 C CNN
-F 2 "Button_Switch_SMD:SW_SPST_SKQG_WithStem" H 5900 2550 50  0001 C CNN
+F 2 "Button_SMD:SW_SPST_SKQG_WithStem" H 5900 2550 50  0001 C CNN
 F 3 "~" H 5900 2550 50  0001 C CNN
+F 4 "C318887" H 5900 2350 50  0001 C CNN "LCSC_ID"
 	1    5900 2350
 	1    0    0    -1
@@
 F 2 "Resistor_SMD:R_0603_1608Metric" V 4580 2350 50  0001 C CNN
 F 3 "~" H 4650 2350 50  0001 C CNN
+F 4 "C4190" H 4650 2350 50  0001 C CNN "LCSC_ID"
 	1    4650 2350
 	0    -1   -1   0
@@
 F 2 "Capacitor_SMD:C_0603_1608Metric" H 5238 2450 50  0001 C CNN
 F 3 "~" H 5200 2600 50  0001 C CNN
+F 4 "C14663" H 5200 2600 50  0001 C CNN "LCSC_ID"
 	1    5200 2600
 	1    0    0    -1
@@
 F 0 "SW3" H 5900 3885 50  0000 C CNN
 F 1 "SW_Push_Dual_x2" H 5900 3794 50  0000 C CNN
-F 2 "Resistor_SMD:R_0603_1608Metric" H 5900 3800 50  0001 C CNN
+F 2 "Button_SMD:SW_SPST_SKQG_WithStem" H 5900 3800 50  0001 C CNN
 F 3 "~" H 5900 3800 50  0001 C CNN
+F 4 "C318887" H 5900 3600 50  0001 C CNN "LCSC_ID"
 	1    5900 3600
 	1    0    0    -1
@@
 F 2 "Resistor_SMD:R_0603_1608Metric" V 4580 3600 50  0001 C CNN
 F 3 "~" H 4650 3600 50  0001 C CNN
+F 4 "C4190" H 4650 3600 50  0001 C CNN "LCSC_ID"
 	1    4650 3600
 	0    -1   -1   0
@@
 F 2 "Capacitor_SMD:C_0603_1608Metric" H 5238 3700 50  0001 C CNN
 F 3 "~" H 5200 3850 50  0001 C CNN
+F 4 "C14663" H 5200 3850 50  0001 C CNN "LCSC_ID"
 	1    5200 3850
 	1    0    0    -1
@@
 F 0 "SW2" H 5900 5185 50  0000 C CNN
 F 1 "SW_Push_Dual_x2" H 5900 5094 50  0000 C CNN
-F 2 "Button_Switch_SMD:SW_SPST_SKQG_WithStem" H 5900 5100 50  0001 C CNN
+F 2 "Button_SMD:SW_SPST_SKQG_WithStem" H 5900 5100 50  0001 C CNN
 F 3 "~" H 5900 5100 50  0001 C CNN
+F 4 "C318887" H 5900 4900 50  0001 C CNN "LCSC_ID"
 	1    5900 4900
 	1    0    0    -1
@@
 F 2 "Resistor_SMD:R_0603_1608Metric" V 4580 4900 50  0001 C CNN
 F 3 "~" H 4650 4900 50  0001 C CNN
+F 4 "C4190" H 4650 4900 50  0001 C CNN "LCSC_ID"
 	1    4650 4900
 	0    -1   -1   0
@@
 F 2 "Capacitor_SMD:C_0603_1608Metric" H 5238 5000 50  0001 C CNN
 F 3 "~" H 5200 5150 50  0001 C CNN
+F 4 "C14663" H 5200 5150 50  0001 C CNN "LCSC_ID"
 	1    5200 5150
 	1    0    0    -1

Commit message: Routing schema
Parts:
- removed C3: 100n, Capacitor_SMD:C_0603_1608Metric, symbol Device:C
- removed R3: 2k2, Resistor_SMD:R_0603_1608Metric, symbol Device:R
- removed SW2: SW_Push_Dual_x2, Button_SMD:SW_SPST_SKQG_WithStem, symbol Switch:SW_Push_Dual_x2
Changed lines of the file:
@@
-	1    0    0    -1
-$EndComp
-$Comp
-L Switch:SW_Push_Dual_x2 SW?
-U 1 1 5F8CFBA7
-P 5900 4900
-AR Path="/5F8CFBA7" Ref="SW?"  Part="1"
-AR Path="/5F8BD394/5F8CFBA7" Ref="SW2"  Part="1"
-F 0 "SW2" H 5900 5185 50  0000 C CNN
-F 1 "SW_Push_Dual_x2" H 5900 5094 50  0000 C CNN
-F 2 "Button_SMD:SW_SPST_SKQG_WithStem" H 5900 5100 50  0001 C CNN
-F 3 "~" H 5900 5100 50  0001 C CNN
-F 4 "C318887" H 5900 4900 50  0001 C CNN "LCSC_ID"
-	1    5900 4900
-	1    0    0    -1
-$EndComp
-Wire Wire Line
-	5700 4900 5200 4900
-Text HLabel 4350 4900 0    50   Input ~ 0
-BTN_2
-$Comp
-L Device:R R3
-U 1 1 5F8CFBAF
-P 4650 4900
-F 0 "R3" V 4857 4900 50  0000 C CNN
-F 1 "2k2" V 4766 4900 50  0000 C CNN
-F 2 "Resistor_SMD:R_0603_1608Metric" V 4580 4900 50  0001 C CNN
-F 3 "~" H 4650 4900 50  0001 C CNN
-F 4 "C4190" H 4650 4900 50  0001 C CNN "LCSC_ID"
-	1    4650 4900
-	0    -1   -1   0
-$EndComp
-Wire Wire Line
-	4500 4900 4350 4900
-Wire Wire Line
-	5200 4900 5200 5000
-Connection ~ 5200 4900
-Wire Wire Line
-	5200 4900 4800 4900
-$Comp
-L Device:C C3
-U 1 1 5F8CFBB9
-P 5200 5150
-F 0 "C3" H 5315 5196 50  0000 L CNN
-F 1 "100n" H 5315 5105 50  0000 L CNN
-F 2 "Capacitor_SMD:C_0603_1608Metric" H 5238 5000 50  0001 C CNN
-F 3 "~" H 5200 5150 50  0001 C CNN
-F 4 "C14663" H 5200 5150 50  0001 C CNN "LCSC_ID"
-	1    5200 5150
-	1    0    0    -1
-$EndComp
-Wire Wire Line
-	5200 5300 5200 5400
-Wire Wire Line
-	5200 5400 6250 5400
-Wire Wire Line
-	6250 5400 6250 4900
-Wire Wire Line
-	6250 4900 6100 4900
-Wire Wire Line
-	6250 5400 6250 5500
-Connection ~ 6250 5400
-$Comp
-L power:GND #PWR0107
-U 1 1 5F8CFBC5
-P 6250 5500
-F 0 "#PWR0107" H 6250 5250 50  0001 C CNN
-F 1 "GND" H 6255 5327 50  0000 C CNN
-F 2 "" H 6250 5500 50  0001 C CNN
-F 3 "" H 6250 5500 50  0001 C CNN
-	1    6250 5500
 	1    0    0    -1
 $EndComp

Commit message: Routing board
Parts:
- SW1: value SW_Push_Dual_x2 -> Reset_Button
- SW3: value SW_Push_Dual_x2 -> User_Button
Changed lines of the file:
@@
 AR Path="/5F8BD394/5F8BE17E" Ref="SW1"  Part="1"
 F 0 "SW1" H 5900 2635 50  0000 C CNN
-F 1 "SW_Push_Dual_x2" H 5900 2544 50  0000 C CNN
+F 1 "Reset_Button" H 5900 2544 50  0000 C CNN
 F 2 "Button_SMD:SW_SPST_SKQG_WithStem" H 5900 2550 50  0001 C CNN
 F 3 "~" H 5900 2550 50  0001 C CNN
@@
 AR Path="/5F8BD394/5F8CDCBE" Ref="SW3"  Part="1"
 F 0 "SW3" H 5900 3885 50  0000 C CNN
-F 1 "SW_Push_Dual_x2" H 5900 3794 50  0000 C CNN
+F 1 "User_Button" H 5900 3794 50  0000 C CNN
 F 2 "Button_SMD:SW_SPST_SKQG_WithStem" H 5900 3800 50  0001 C CNN
 F 3 "~" H 5900 3800 50  0001 C CNN
