File: hw/Pletacka-board.sch (KiCad schematic (older format))
At the start: 37 parts, among them J4 STOP_INPUT, J5 POWER_&_FINN_INPUT, SW1 Reset_Button, SW2 User_Button, U1 TPS54231D, U2 EL357N(A)(TA)-G, U3 EL357N(A)(TA)-G

Commit message: Testin fabrication export
Parts:
- C1: LCSC (none) -> C13585; LCSC_ID C13585 -> (none)
- C2: LCSC (none) -> C21117; LCSC_ID C21117 -> (none)
- C3: LCSC (none) -> C21122; LCSC_ID C21122 -> (none)
- C4: LCSC (none) -> C1032; LCSC_ID C1032 -> (none)
- C5, C7, C8: LCSC (none) -> C14663; LCSC_ID C14663 -> (none)
- C6: LCSC (none) -> C45783; LCSC_ID C45783 -> (none)
- D1, D5: LCSC (none) -> C8678; LCSC_ID C8678 -> (none)
- D2: LCSC (none) -> C49827; LCSC_ID C49827 -> (none)
- D3: LCSC (none) -> C72043; LCSC_ID C72043 -> (none)
- D4: LCSC (none) -> C2286; LCSC_ID C2286 -> (none)
- D6, D7: LCSC (none) -> C8598; LCSC_ID C8598 -> (none)
- L1: LCSC (none) -> C206321; LCSC_ID C206321 -> (none)
- POLYFUSE1: LCSC (none) -> C70076; LCSC_ID C70076 -> (none)
- R1, R2, R8, R9: LCSC (none) -> C4190; LCSC_ID C4190 -> (none)
- R10, R11: LCSC (none) -> C25804; LCSC_ID C25804 -> (none)
- R3: LCSC (none) -> C22775; LCSC_ID C22775 -> (none)
- R4: LCSC (none) -> C23162; LCSC_ID C23162 -> (none)
- R5: LCSC (none) -> C22809; LCSC_ID C22809 -> (none)
- R6, R7: LCSC (none) -> C4184; LCSC_ID C4184 -> (none)
- SW1, SW2: LCSC (none) -> C620322; LCSC_ID C620322 -> (none)
- U1: LCSC (none) -> C9865; LCSC_ID C9865 -> (none)
- U2, U3: LCSC (none) -> C6649; LCSC_ID C6649 -> (none)
Changed lines of the file:
@@
 F 2 "Button_SMD:Button_SMD_10mm" H 10300 1500 50  0001 C CNN
 F 3 "~" H 10300 1500 50  0001 C CNN
-F 4 "C620322" H 10300 1300 50  0001 C CNN "LCSC_ID"
+F 4 "C620322" H 10300 1300 50  0001 C CNN "LCSC"
 	1    10300 1300
 	1    0    0    -1
@@
 F 2 "Resistor_SMD:R_0603_1608Metric" V 8980 1300 50  0001 C CNN
 F 3 "~" H 9050 1300 50  0001 C CNN
-F 4 "C4190" H 9050 1300 50  0001 C CNN "LCSC_ID"
+F 4 "C4190" H 9050 1300 50  0001 C CNN "LCSC"
 	1    9050 1300
 	0    -1   -1   0
@@
 F 2 "Capacitor_SMD:C_0603_1608Metric" H 9638 1400 50  0001 C CNN
 F 3 "~" H 9600 1550 50  0001 C CNN
-F 4 "C14663" H 9600 1550 50  0001 C CNN "LCSC_ID"
+F 4 "C14663" H 9600 1550 50  0001 C CNN "LCSC"
 	1    9600 1550
 	1    0    0    -1
@@
 F 2 "Button_SMD:Button_SMD_10mm" H 10300 2450 50  0001 C CNN
 F 3 "~" H 10300 2450 50  0001 C CNN
-F 4 "C620322" H 10300 2250 50  0001 C CNN "LCSC_ID"
+F 4 "C620322" H 10300 2250 50  0001 C CNN "LCSC"
 	1    10300 2250
 	1    0    0    -1
@@
 F 2 "Resistor_SMD:R_0603_1608Metric" V 8980 2250 50  0001 C CNN
 F 3 "~" H 9050 2250 50  0001 C CNN
-F 4 "C4190" H 9050 2250 50  0001 C CNN "LCSC_ID"
+F 4 "C4190" H 9050 2250 50  0001 C CNN "LCSC"
 	1    9050 2250
 	0    -1   -1   0
@@
 F 2 "Capacitor_SMD:C_0603_1608Metric" H 9638 2350 50  0001 C CNN
 F 3 "~" H 9600 2500 50  0001 C CNN
-F 4 "C14663" H 9600 2500 50  0001 C CNN "LCSC_ID"
+F 4 "C14663" H 9600 2500 50  0001 C CNN "LCSC"
 	1    9600 2500
 	1    0    0    -1
@@
 F 2 "B5819W:B5819W_SOD-123" H 8600 4500 50  0001 L BNN
 F 3 "" H 8600 4500 50  0001 C CNN
-F 4 "C8598" V 8600 4500 50  0001 C CNN "LCSC_ID"
+F 4 "C8598" V 8600 4500 50  0001 C CNN "LCSC"
 	1    8600 4500
 	0    -1   -1   0
@@
 F 2 "Resistor_SMD:R_0603_1608Metric" V 7930 4450 50  0001 C CNN
 F 3 "~" H 8000 4450 50  0001 C CNN
-F 4 "C4184" V 8000 4450 50  0001 C CNN "LCSC_ID"
+F 4 "C4184" V 8000 4450 50  0001 C CNN "LCSC"
 	1    8000 4450
 	0    1    1    0
@@
 F 2 "Resistor_SMD:R_0603_1608Metric" V 10308 4130 39  0001 C CNN
 F 3 "~" H 10400 4150 50  0001 C CNN
-F 4 "C25804" H 10400 4150 50  0001 C CNN "LCSC_ID"
+F 4 "C25804" H 10400 4150 50  0001 C CNN "LCSC"
 	1    10400 4150
 	1    0    0    -1
@@
 F 2 "B5819W:B5819W_SOD-123" H 8600 5850 50  0001 L BNN
 F 3 "" H 8600 5850 50  0001 C CNN
-F 4 "C8598" V 8600 5850 50  0001 C CNN "LCSC_ID"
+F 4 "C8598" V 8600 5850 50  0001 C CNN "LCSC"
 	1    8600 5850
 	0    -1   -1   0
@@
 F 2 "Resistor_SMD:R_0603_1608Metric" V 7930 5800 50  0001 C CNN
 F 3 "~" H 8000 5800 50  0001 C CNN
-F 4 "C4184" V 8000 5800 50  0001 C CNN "LCSC_ID"
+F 4 "C4184" V 8000 5800 50  0001 C CNN "LCSC"
 	1    8000 5800
 	0    1    1    0
@@
 F 2 "Resistor_SMD:R_0603_1608Metric" V 10330 5500 50  0001 C CNN
 F 3 "~" H 10400 5500 50  0001 C CNN
-F 4 "C25804" H 10400 5500 50  0001 C CNN "LCSC_ID"
+F 4 "C25804" H 10400 5500 50  0001 C CNN "LCSC"
 	1    10400 5500
 	1    0    0    -1
@@
 F 3 "https://www.snapeda.com/parts/EL357N(A)(TA)-G/Everlight%20Electronics/datasheet/" H 9600 5850 50  0001 L BNN
 F 4 "https://www.snapeda.com/parts/EL357N%28A%29%28TA%29-G/Everlight%20Electronics/view-part/?ref=search&t=EL357N(A)(TA)-G" H 9900 5300 50  0001 C CNN "Source"
-F 5 "C6649" H 9600 5150 50  0001 C CNN "LCSC_ID"
+F 5 "C6649" H 9600 5150 50  0001 C CNN "LCSC"
 	1    9600 5850
 	1    0    0    -1
@@
 F 3 "https://www.snapeda.com/parts/EL357N(A)(TA)-G/Everlight%20Electronics/datasheet/" H 9600 4500 50  0001 L BNN
 F 4 "https://www.snapeda.com/parts/EL357N%28A%29%28TA%29-G/Everlight%20Electronics/view-part/?ref=search&t=EL357N(A)(TA)-G" H 9900 3950 50  0001 C CNN "Source"
-F 5 "C6649" H 9600 3800 50  0001 C CNN "LCSC_ID"
+F 5 "C6649" H 9600 3800 50  0001 C CNN "LCSC"
 	1    9600 4500
 	1    0    0    -1
@@
 F 2 "Resistor_SMD:R_1206_3216Metric" V 1780 1200 50  0001 C CNN
 F 3 "~" H 1850 1200 50  0001 C CNN
-F 4 "C70076" V 1850 1200 50  0001 C CNN "LCSC_ID"
+F 4 "C70076" V 1850 1200 50  0001 C CNN "LCSC"
 	1    1850 1200
 	0    -1   -1   0
@@
 F 2 "Capacitor_SMD:C_1206_3216Metric" H 2538 1700 50  0001 C CNN
 F 3 "~" H 2500 1850 50  0001 C CNN
-F 4 "C13585" H 2500 1850 50  0001 C CNN "LCSC_ID"
+F 4 "C13585" H 2500 1850 50  0001 C CNN "LCSC"
 	1    2500 1850
 	1    0    0    -1
@@
 F 3 "https://www.snapeda.com/parts/1SMB5935BT3G/ON%20Semiconductor/datasheet/" H 2200 1400 50  0001 L BNN
 F 4 "https://snapeda.com/shop?store=Arrow+Electronics&id=285964" H 2350 1050 50  0001 C CNN "Source"
-F 5 "C49827" V 2200 1400 50  0001 C CNN "LCSC_ID"
+F 5 "C49827" V 2200 1400 50  0001 C CNN "LCSC"
 	1    2200 1400
 	0    -1   -1   0
@@
 F 3 "https://www.snapeda.com/parts/TPS54231D/Texas%20Instruments/datasheet/" H 4600 1900 50  0001 C CNN
 F 4 "https://www.snapeda.com/parts/TPS54231D/Texas%20Instruments/view-part/?ref=search&t=TPS54231" H 4650 700 50  0001 C CNN "Source"
-F 5 "C9865" H 4600 1900 50  0001 C CNN "LCSC_ID"
+F 5 "C9865" H 4600 1900 50  0001 C CNN "LCSC"
 	1    4600 1900
 	1    0    0    -1
@@
 F 2 "Capacitor_SMD:C_0603_1608Metric" H 3588 2550 50  0001 C CNN
 F 3 "~" H 3550 2700 50  0001 C CNN
-F 4 "C1032" H 3550 2700 50  0001 C CNN "LCSC_ID"
+F 4 "C1032" H 3550 2700 50  0001 C CNN "LCSC"
 	1    3550 2700
 	1    0    0    -1
@@
 F 2 "Capacitor_SMD:C_0603_1608Metric" H 3238 2550 50  0001 C CNN
 F 3 "~" H 3200 2700 50  0001 C CNN
-F 4 "C21122" H 3200 2700 50  0001 C CNN "LCSC_ID"
+F 4 "C21122" H 3200 2700 50  0001 C CNN "LCSC"
 	1    3200 2700
 	1    0    0    -1
@@
 F 2 "Capacitor_SMD:C_0603_1608Metric" H 2838 2550 50  0001 C CNN
 F 3 "~" H 2800 2700 50  0001 C CNN
-F 4 "C21117" H 2800 2700 50  0001 C CNN "LCSC_ID"
+F 4 "C21117" H 2800 2700 50  0001 C CNN "LCSC"
 	1    2800 2700
 	1    0    0    -1
@@
 F 2 "Resistor_SMD:R_0603_1608Metric" V 3130 2050 50  0001 C CNN
 F 3 "~" H 3200 2050 50  0001 C CNN
-F 4 "C22775" H 3200 2050 50  0001 C CNN "LCSC_ID"
+F 4 "C22775" H 3200 2050 50  0001 C CNN "LCSC"
 	1    3200 2050
 	1    0    0    -1
@@
 F 3 "https://www.snapeda.com/parts/SS34/ON%20Semiconductor/datasheet/" H 1350 1200 50  0001 L BNN
 F 4 "https://www.snapeda.com/parts/SS34/ON%20Semiconductor/view-part/?ref=search&t=SS34" H 1300 850 50  0001 C CNN "Source"
-F 5 "C8678" H 1350 1200 50  0001 C CNN "LCSC_ID"
+F 5 "C8678" H 1350 1200 50  0001 C CNN "LCSC"
 	1    1350 1200
 	1    0    0    -1
@@
 F 3 "https://www.snapeda.com/parts/SS34/ON%20Semiconductor/datasheet/" H 5850 1750 50  0001 L BNN
 F 4 "https://www.snapeda.com/parts/SS34/ON%20Semiconductor/view-part/?ref=search&t=SS34" H 5800 1400 50  0001 C CNN "Source"
-F 5 "C8678" H 5850 1750 50  0001 C CNN "LCSC_ID"
+F 5 "C8678" H 5850 1750 50  0001 C CNN "LCSC"
 	1    5850 1750
 	0    1    1    0
@@
 F 3 "~" H 5450 1750 50  0001 C CNN
 F 4 "" H 5450 1750 50  0001 C CNN "LSCS_ID"
-F 5 "C14663" H 5450 1750 50  0001 C CNN "LCSC_ID"
+F 5 "C14663" H 5450 1750 50  0001 C CNN "LCSC"
 	1    5450 1750
 	1    0    0    -1
@@
 F 2 "Resistor_SMD:R_0603_1608Metric" V 6530 2400 50  0001 C CNN
 F 3 "~" H 6600 2400 50  0001 C CNN
-F 4 "C23162" H 6600 2400 50  0001 C CNN "LCSC_ID"
+F 4 "C23162" H 6600 2400 50  0001 C CNN "LCSC"
 	1    6600 2400
 	1    0    0    -1
@@
 F 2 "Resistor_SMD:R_0603_1608Metric" V 6530 2950 50  0001 C CNN
 F 3 "~" H 6600 2950 50  0001 C CNN
-F 4 "C22809" H 6600 2950 50  0001 C CNN "LCSC_ID"
+F 4 "C22809" H 6600 2950 50  0001 C CNN "LCSC"
 	1    6600 2950
 	1    0    0    -1
@@
 F 2 "Capacitor_SMD:C_0603_1608Metric" H 6988 2500 50  0001 C CNN
 F 3 "~" H 6950 2650 50  0001 C CNN
-F 4 "C45783" H 6950 2650 50  0001 C CNN "LCSC_ID"
+F 4 "C45783" H 6950 2650 50  0001 C CNN "LCSC"
 	1    6950 2650
 	1    0    0    -1
@@
 F 2 "SLW6045S220MST:SLW" H 6200 2100 50  0001 C CNN
 F 3 "~" H 6200 2100 50  0001 C CNN
-F 4 "C206321" V 6200 2100 50  0001 C CNN "LCSC_ID"
+F 4 "C206321" V 6200 2100 50  0001 C CNN "LCSC"
 	1    6200 2100
 	0    -1   -1   0
@@
 F 2 "Resistor_SMD:R_0603_1608Metric" V 2080 4750 50  0001 C CNN
 F 3 "~" H 2150 4750 50  0001 C CNN
-F 4 "C4190" H 2150 4750 50  0001 C CNN "LCSC_ID"
+F 4 "C4190" H 2150 4750 50  0001 C CNN "LCSC"
 	1    2150 4750
 	0    1    1    0
@@
 F 2 "LED_SMD:LED_0603_1608Metric" H 2700 4750 50  0001 C CNN
 F 3 "~" H 2700 4750 50  0001 C CNN
-F 4 "C2286" H 2700 4750 50  0001 C CNN "LCSC_ID"
+F 4 "C2286" H 2700 4750 50  0001 C CNN "LCSC"
 	1    2700 4750
 	-1   0    0    1
@@
 F 2 "Resistor_SMD:R_0603_1608Metric" V 2080 4150 50  0001 C CNN
 F 3 "~" H 2150 4150 50  0001 C CNN
-F 4 "C4190" H 2150 4150 50  0001 C CNN "LCSC_ID"
+F 4 "C4190" H 2150 4150 50  0001 C CNN "LCSC"
 	1    2150 4150
 	0    1    1    0
@@
 F 2 "LED_SMD:LED_0603_1608Metric" H 2700 4150 50  0001 C CNN
 F 3 "~" H 2700 4150 50  0001 C CNN
-F 4 "C72043" H 2700 4150 50  0001 C CNN "LCSC_ID"
+F 4 "C72043" H 2700 4150 50  0001 C CNN "LCSC"
 	1    2700 4150
 	-1   0    0    1

Commit message: Finish board
Parts:
- added JP1: Jumper_NO_Small, Jumper:SolderJumper-2_P1.3mm_Open_Pad1.0x1.5mm, symbol Device:Jumper_NO_Small
- added JP2: Jumper, Jumper:SolderJumper-2_P1.3mm_Bridged_Pad1.0x1.5mm, symbol Device:Jumper
- added Pins1: Pins, Connector_PinHeader_2.54mm:PinHeader_1x05_P2.54mm_Vertical, symbol Connector:Conn_01x05_Female
- renumbered E1 to ESP1, H1 to MHole1, J5 to POWER_&_FINN_INPUT1, J4 to STOP_INPUT1
Connections:
- net labels added: USER_IO25, USER_IO33
- wire segments 129 -> 138
Other:
- note added: "Pins"
Changed lines of the file:
@@
 OPTO_STOP
 $Comp
-L Connector:Conn_01x02_Female J4
+L Connector:Conn_01x02_Female STOP_INPUT1
 U 1 1 5F9151EB
 P 1300 5650
-F 0 "J4" V 1238 5462 50  0000 R CNN
+F 0 "STOP_INPUT1" V 1238 5462 50  0000 R CNN
 F 1 "STOP_INPUT" V 1147 5462 50  0000 R CNN
 F 2 "Terminal_block:TerminalBlock_Phoenix_PT-1,5-2-5.0-H_1x02_P5.00mm_Horizontal" H 1300 5650 50  0001 C CNN
@@
 $EndComp
 $Comp
-L Connector:Conn_01x03_Female J5
+L Connector:Conn_01x03_Female POWER_&_FINN_INPUT1
 U 1 1 5F915FED
 P 2450 5650
-F 0 "J5" V 2388 5462 50  0000 R CNN
+F 0 "POWER_&_FINN_INPUT1" V 2388 5462 50  0000 R CNN
 F 1 "POWER_&_FINN_INPUT" V 2297 5462 50  0000 R CNN
 F 2 "Terminal_block:TerminalBlock_Phoenix_PT-1,5-3-5.0-H_1x03_P5.00mm_Horizontal" H 2450 5650 50  0001 C CNN
@@
 Input
 $Comp
-L Mechanical:MountingHole H1
+L Mechanical:MountingHole MHole1
 U 1 1 5F9A042D
 P 6200 7600
-F 0 "H1" H 6300 7646 50  0000 L CNN
+F 0 "MHole1" H 6300 7646 50  0000 L CNN
 F 1 "MountingHole" H 6300 7555 50  0000 L CNN
 F 2 "MountingHole:MountingHole_2.7mm_M2.5_Pad" H 6200 7600 50  0001 C CNN
@@
 	6950 3150 6600 3150
 Connection ~ 6600 3150
-Wire Wire Line
-	6950 2100 7250 2100
-Connection ~ 6950 2100
 $Comp
 L power:+3V3 #PWR?
 U 1 1 5F957882
-P 7250 2100
+P 7650 2100
 AR Path="/5F8F7408/5F957882" Ref="#PWR?"  Part="1"
 AR Path="/5F957882" Ref="#PWR0114"  Part="1"
-F 0 "#PWR0114" H 7250 1950 50  0001 C CNN
-F 1 "+3V3" V 7265 2228 50  0000 L CNN
-F 2 "" H 7250 2100 50  0001 C CNN
-F 3 "" H 7250 2100 50  0001 C CNN
-	1    7250 2100
+F 0 "#PWR0114" H 7650 1950 50  0001 C CNN
+F 1 "+3V3" V 7750 1950 50  0000 L CNN
+F 2 "" H 7650 2100 50  0001 C CNN
+F 3 "" H 7650 2100 50  0001 C CNN
+	1    7650 2100
 	0    1    1    0
 $EndComp
@@
 	3200 1600 3900 1600
 Wire Notes Line
-	650  750  7650 750
-Wire Notes Line
-	7650 750  7650 3400
-Wire Notes Line
-	7650 3400 650  3400
+	650  750  7800 750
+Wire Notes Line
+	7800 750  7800 3400
+Wire Notes Line
+	7800 3400 650  3400
 Wire Notes Line
 	650  3400 650  750
@@
 Text GLabel 5550 6650 2    50   Input ~ 0
 BTN_RESET
-Text GLabel 5550 6550 2    50   Input ~ 0
+Text GLabel 5550 6350 2    50   Input ~ 0
 BTN_USER
 Wire Wire Line
@@
 $EndComp
 $Comp
-L ESP32-TTGO-T-Display:ESP32-TTGO-T-Display E1
+L ESP32-TTGO-T-Display:ESP32-TTGO-T-Display ESP1
 U 1 1 5F8A9387
 P 4850 6300
-F 0 "E1" H 4945 6875 50  0000 C CNN
+F 0 "ESP1" H 4945 6875 50  0000 C CNN
 F 1 "ESP32-TTGO-T-Display" H 4945 6784 50  0000 C CNN
 F 2 "ESP32-TTGO-T-Display:ESP32-TTGO-T-Display" H 3850 6750 50  0001 C CNN
@@
 Text Notes 2450 4950 0    79   ~ 0
 User LED
+Text GLabel 5550 6550 2    50   Input ~ 0
+USER_IO25
+Text GLabel 5550 6450 2    50   Input ~ 0
+USER_IO33
+$Comp
+L Connector:Conn_01x05_Female Pins1
+U 1 1 5F918B43
+P 4900 4000
+F 0 "Pins1" V 4838 3712 50  0000 R CNN
+F 1 "Pins" V 4747 3712 50  0000 R CNN
+F 2 "Connector_PinHeader_2.54mm:PinHeader_1x05_P2.54mm_Vertical" H 4900 4000 50  0001 C CNN
+F 3 "~" H 4900 4000 50  0001 C CNN
+	1    4900 4000
+	0    -1   -1   0
+$EndComp
+Wire Wire Line
+	5100 4200 5100 4400
+Wire Wire Line
+	5000 4200 5000 4400
+Wire Wire Line
+	4900 4200 4900 4400
+Wire Wire Line
+	4800 4200 4800 4400
+Wire Wire Line
+	4700 4200 4700 4400
+$Comp
+L power:GND #PWR0120
+U 1 1 5F9547E1
+P 4900 4400
+F 0 "#PWR0120" H 4900 4150 50  0001 C CNN
+F 1 "GND" V 4905 4272 50  0000 R CNN
+F 2 "" H 4900 4400 50  0001 C CNN
+F 3 "" H 4900 4400 50  0001 C CNN
+	1    4900 4400
+	1    0    0    -1
+$EndComp
+$Comp
+L power:+3V3 #PWR0121
+U 1 1 5F955A16
+P 5100 4400
+F 0 "#PWR0121" H 5100 4250 50  0001 C CNN
+F 1 "+3V3" V 5115 4528 50  0000 L CNN
+F 2 "" H 5100 4400 50  0001 C CNN
+F 3 "" H 5100 4400 50  0001 C CNN
+	1    5100 4400
+	-1   0    0    1
+$EndComp
+$Comp
+L power:+5V #PWR0122
+U 1 1 5F95698D
+P 4700 4400
+F 0 "#PWR0122" H 4700 4250 50  0001 C CNN
+F 1 "+5V" V 4715 4528 50  0000 L CNN
+F 2 "" H 4700 4400 50  0001 C CNN
+F 3 "" H 4700 4400 50  0001 C CNN
+	1    4700 4400
+	-1   0    0    1
+$EndComp
+Text GLabel 4800 4400 3    50   Input ~ 0
+USER_IO25
+Text GLabel 5000 4400 3    50   Input ~ 0
+USER_IO33
+Wire Wire Line
+	6950 2100 7050 2100
+Connection ~ 6950 2100
+Wire Notes Line
+	4350 3900 5600 3900
+Wire Notes Line
+	5600 3900 5600 5050
+Wire Notes Line
+	5600 5050 4350 5050
+Wire Notes Line
+	4350 5050 4350 3900
+Text Notes 4700 3900 0    197  ~ 0
+Pins
+Wire Wire Line
+	2200 1200 2200 850
+Wire Wire Line
+	2200 850  6600 850
+Wire Wire Line
+	6600 850  6600 1300
+Wire Wire Line
+	6600 1300 6800 1300
+$Comp
+L Device:Jumper_NO_Small JP1
+U 1 1 5FAEDA72
+P 6900 1300
+F 0 "JP1" H 6900 1485 50  0000 C CNN
+F 1 "Jumper_NO_Small" H 6900 1394 50  0000 C CNN
+F 2 "Jumper:SolderJumper-2_P1.3mm_Open_Pad1.0x1.5mm" H 6900 1300 50  0001 C CNN
+F 3 "~" H 6900 1300 50  0001 C CNN
+	1    6900 1300
+	1    0    0    -1
+$EndComp
+$Comp
+L power:+5V #PWR0123
+U 1 1 5FAEEF87
+P 7000 1300
+F 0 "#PWR0123" H 7000 1150 50  0001 C CNN
+F 1 "+5V" V 7015 1428 50  0000 L CNN
+F 2 "" H 7000 1300 50  0001 C CNN
+F 3 "" H 7000 1300 50  0001 C CNN
+	1    7000 1300
+	0    1    1    0
+$EndComp
+$Comp
+L Device:Jumper JP2
+U 1 1 5FAF5BD0
+P 7350 2100
+F 0 "JP2" H 7350 2364 50  0000 C CNN
+F 1 "Jumper" H 7350 2273 50  0000 C CNN
+F 2 "Jumper:SolderJumper-2_P1.3mm_Bridged_Pad1.0x1.5mm" H 7350 2100 50  0001 C CNN
+F 3 "~" H 7350 2100 50  0001 C CNN
+	1    7350 2100
+	1    0    0    -1
+$EndComp
 $EndSCHEMATC
