File: Pletacka-board-v1.0/hw/Pletacka_board.brd (EAGLE design)
At the start: 75 x 60 mm, 59 parts, among them U2 EL357N(A)(TA)-G, U3 EL357N(A)(TA)-G, U4 EL357N(A)(TA)-G, U5 EL357N(A)(TA)-G, U6 TPS54231D

Commit message: Nice schema
Parts:
- moved R13 289.9 mm to (15.2, -270.5), turned to 0 degrees
- moved R12 286.1 mm to (10.2, -270.5)
- moved D4 284.2 mm to (1.27, -270.5)
- moved U5 282.0 mm to (3.81, -262.9), turned to 0 degrees
- moved R11 263.3 mm to (15.2, -243.8), turned to 0 degrees
- moved CON4 261.2 mm to (5.08, -254.0)
- moved R10 259.7 mm to (10.2, -243.8)
- moved D2 258.4 mm to (1.27, -243.8)
- moved U4 256.1 mm to (3.81, -236.2), turned to 0 degrees
- moved R9 238.8 mm to (0.00, -217.2), turned to 0 degrees
- moved CON3 235.2 mm to (5.08, -227.3)
- moved R7 231.8 mm to (15.2, -210.8), turned to 0 degrees
- moved D6 228.8 mm to (1.27, -210.8)
- moved R6 228.7 mm to (10.2, -210.8)
- moved R8 226.7 mm to (20.3, -210.8)
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Routing:
- net +3V3: track 158.5 -> 69.3 mm
- net +5V: track 87.7 -> 5.39 mm
- net TMP_SDA: track 46.3 -> 0.00 mm
- net TMP_SCL: track 45.4 -> 0.00 mm
- net +24V: track 42.9 -> 0.00 mm
- net OPTO4: track 37.3 -> 0.00 mm
- net TMP_OS: track 36.0 -> 0.00 mm
- net OPTO3: track 31.3 -> 0.00 mm
- net GND: track 86.6 -> 63.3 mm, vias 14 -> 11
- net OPTO2: track 22.5 -> 0.00 mm
- net BOOT: track 16.2 -> 0.00 mm, vias 2 -> 0
- net OPTO1: track 15.2 -> 0.00 mm
- net VSENSE: track 11.1 -> 0.00 mm
- net N$17: track 9.22 -> 0.00 mm
- net N$16: track 9.19 -> 0.00 mm
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